Commit message: simulation control added

File: description/robot_core.xacro (robot description, xacro)
@@ -41,4 +41,7 @@
         </xacro:inertial_box>
     </link>
+    <gazebo reference="chassis">
+        <material>Gazebo/White</material>
+    </gazebo>
 <!-- LEFT DRIVE WHEEL LINK -->
     <joint name="left_wheel_joint" type="continuous">
@@ -64,4 +67,7 @@
         </xacro:inertial_cylinder>
     </link>
+    <gazebo reference="left_wheel">
+        <material>Gazebo/Orange</material>
+    </gazebo>
 <!-- RIGHT DRIVE WHEEL LINK -->
 <joint name="right_wheel_joint" type="continuous">
@@ -87,4 +93,7 @@
     </xacro:inertial_cylinder>
 </link>
+<gazebo reference="right_wheel">
+    <material>Gazebo/Orange</material>
+</gazebo>
 <!-- LEFT DUMMY WHEEL LINK -->
 <joint name="left_dummywheel_joint" type="fixed">
@@ -109,4 +118,9 @@
     </xacro:inertial_cylinder>
 </link>
+<gazebo reference="left_dummywheel">
+    <material>Gazebo/Orange</material>
+    <mu1 value="0.0001"/>
+    <mu2 value="0.0001"/>
+</gazebo>
 <!-- RIGHT DUMMY WHEEL LINK -->
 <joint name="right_dummywheel_joint" type="fixed">
@@ -131,3 +145,8 @@
     </xacro:inertial_cylinder>
 </link>
+<gazebo reference="right_dummywheel">
+    <material>Gazebo/Orange</material>
+    <mu1 value="0.0001"/>
+    <mu2 value="0.0001"/>
+</gazebo>
 </robot>
