Commit message: 4 wheel drive implemented

File: description/gazebo_control.xacro (robot description, xacro)
@@ -4,6 +4,11 @@
         <plugin name="diff_drive" filename="libgazebo_ros_diff_drive.so">
             <!-- Wheel Info -->
-            <left_joint>left_wheel_joint</left_joint>
-            <right_joint>right_wheel_joint</right_joint>
+            <num_wheel_pairs>2</num_wheel_pairs>
+            <left_joint>lb_wheel_joint</left_joint>
+            <right_joint>rb_wheel_joint</right_joint>
+            <wheel_separation>0.7</wheel_separation>
+            <wheel_diameter>0.5</wheel_diameter>
+            <left_joint>lf_wheel_joint</left_joint>
+            <right_joint>rf_wheel_joint</right_joint>
             <wheel_separation>0.7</wheel_separation>
             <wheel_diameter>0.5</wheel_diameter>

File: description/robot_core.xacro (robot description, xacro)
@@ -2,4 +2,6 @@
 <robot xmlns:xacro="http://www.ros.org/wiki/xacro" >
     <xacro:include filename="inertial_macros.xacro"/>
+    <!-- friction constant -->
+    <xacro:property name="friction_constant" value="0.2"/>
     <material name="white">
         <color rgba="1 1 1 1"/>
@@ -47,12 +49,13 @@
         <material>Gazebo/White</material>
     </gazebo>
-<!-- LEFT DRIVE WHEEL LINK -->
-    <joint name="left_wheel_joint" type="continuous">
+<!-- BACK LEFT WHEEL LINK -->
+    <joint name="lb_wheel_joint" type="continuous">
         <parent link="base_link"/>
-        <child link="left_wheel"/>
+        <child link="lb_wheel"/>
         <origin xyz="0 0.35 0" rpy="-${pi/2} 0 0"/>
         <axis xyz="0 0 1"/>
+        <limit effort="1000" velocity="1000"/>
     </joint>
-    <link name="left_wheel">
+    <link name="lb_wheel">
         <visual>
             <geometry>
@@ -70,15 +73,18 @@
         </xacro:inertial_cylinder>
     </link>
-    <gazebo reference="left_wheel">
+    <gazebo reference="lb_wheel">
+        <!-- <mu1>${friction_constant}</mu1>
+        <mu2>${friction_constant}</mu2> -->
         <material>Gazebo/Orange</material>
     </gazebo>
-<!-- RIGHT DRIVE WHEEL LINK -->
-<joint name="right_wheel_joint" type="continuous">
+<!-- BACK RIGHT WHEEL LINK -->
+<joint name="rb_wheel_joint" type="continuous">
     <parent link="base_link"/>
-    <child link="right_wheel"/>
+    <child link="rb_wheel"/>
     <origin xyz="0 -0.35 0" rpy="${pi/2} 0 0"/>
     <axis xyz="0 0 -1"/>
+    <limit effort="1000" velocity="1000"/>
 </joint>
-<link name="right_wheel">
+<link name="rb_wheel">
     <visual>
         <geometry>
@@ -96,14 +102,18 @@
     </xacro:inertial_cylinder>
 </link>
-<gazebo reference="right_wheel">
+<gazebo reference="rb_wheel">
+    <!-- <mu1>${friction_constant}</mu1>
+    <mu2>${friction_constant}</mu2> -->
     <material>Gazebo/Orange</material>
 </gazebo>
-<!-- LEFT DUMMY WHEEL LINK -->
-<joint name="left_dummywheel_joint" type="fixed">
-    <parent link="chassis"/>
-    <child link="left_dummywheel"/>
-    <origin xyz="0.95 0.35 0" rpy="-${pi/2} 0 0"/>
+<!-- FRONT LEFT WHEEL LINK -->
+<joint name="lf_wheel_joint" type="continuous">
+    <parent link="base_link"/>
+    <child link="lf_wheel"/>
+    <origin xyz="0.7 0.35 0" rpy="-${pi/2} 0 0"/>
+    <axis xyz="0 0 1"/>
+    <limit effort="1000" velocity="1000"/>
 </joint>
-<link name="left_dummywheel">
+<link name="lf_wheel">
     <visual>
         <geometry>
@@ -121,16 +131,18 @@
     </xacro:inertial_cylinder>
 </link>
-<gazebo reference="left_dummywheel">
+<gazebo reference="lf_wheel">
+    <!-- <mu1>${friction_constant}</mu1>
+    <mu2>${friction_constant}</mu2> -->
     <material>Gazebo/Orange</material>
-    <mu1 value="0.0001"/>
-    <mu2 value="0.0001"/>
 </gazebo>
-<!-- RIGHT DUMMY WHEEL LINK -->
-<joint name="right_dummywheel_joint" type="fixed">
-    <parent link="chassis"/>
-    <child link="right_dummywheel"/>
-    <origin xyz="0.95 -0.35 0" rpy="${pi/2} 0 0"/>
+<!-- FRONT RIGHT WHEEL LINK -->
+<joint name="rf_wheel_joint" type="continuous">
+    <parent link="base_link"/>
+    <child link="rf_wheel"/>
+    <origin xyz="0.7 -0.35 0" rpy="${pi/2} 0 0"/>
+    <axis xyz="0 0 -1"/>
+    <limit effort="1000" velocity="1000"/>
 </joint>
-<link name="right_dummywheel">
+<link name="rf_wheel">
     <visual>
         <geometry>
@@ -148,8 +160,8 @@
     </xacro:inertial_cylinder>
 </link>
-<gazebo reference="right_dummywheel">
+<gazebo reference="rf_wheel">
+    <!-- <mu1>${friction_constant}</mu1>
+    <mu2>${friction_constant}</mu2> -->
     <material>Gazebo/Orange</material>
-    <mu1 value="0.0001"/>
-    <mu2 value="0.0001"/>
 </gazebo>
 </robot>
